File: Hardware/MeshUSB.sch (KiCad schematic (older format))
At the start: 35 parts, among them P1 USB_4, P2 PVCell, Q1 MOS_P, U1 XBEE, U3 LTC3105-MSOP12, U4 FT231X-SSOP, U5 LTC4070

Commit message: Getting moving on v0.2 :)
Changed lines of the file:
@@
 LIBS:ATMega256RFR2
 LIBS:opendous
-LIBS:MeshUSBv0.1-cache
+LIBS:MeshUSB-cache
 EELAYER 24 0
 EELAYER END
@@
 F 3 "" H 1100 5250 60  0000 C CNN
 	1    1100 5250
-	-1   0    0    -1
+	-1   0    0    1
 $EndComp
 $Comp
@@
 NoConn ~ 5150 5450
 Text Notes 8650 700  0    60   ~ 0
-Possible changes for v0.2:\nChange 3105 to 3108 for lower current operation?\nZener diode between usb_vdd and gnd.\n3.3v regulator from power sources to xbee pin 1\nSignaling from 3105 that it is not supplying current\nExternal/high voltage power terminal - traditional PV 6-12v\n  Pull DRV off 4070 to pin for high current charging?\nJumpers for... what needs jumpers? Something must. \n  Charge full indicator? Tx/Rx LEDs? USB vdd?\nSwitch instead of diode isolation for USB/PV power selection?\nUSB Mirrored Insertion Footprint - !Impossible!\nDouble Check Diode footprints - usbvdd is suspect.\nMove battery holder up/change left smt header.\nMove PV connector pins.\nReexamine 10k pullup on #rst. Also supply of LEDs - vccio or usbvdd? Change Rs if necessary change on vccio/usbvdd\nTest points?\nL1 is 0805 package.\nFix problem 0.
+Possible changes for v0.2:\nChange 3105 to 3108 for lower current operation?\nZener diode between usb_vdd and gnd.\n3.3v regulator from power sources to xbee pin 1\nSignaling from 3105 that it is not supplying current\nExternal/high voltage power terminal - traditional PV 6-12v\n  Pull DRV off 4070 to pin for high current charging?\nJumpers for... what needs jumpers? Something must. \n  Charge full indicator? Tx/Rx LEDs? USB vdd?\nSwitch instead of diode isolation for USB/PV power selection? -NO!\nUSB Mirrored Insertion Footprint - !Impossible!\nMove battery holder up/change left smt header.\nMove PV connector pins.\nReexamine 10k pullup on #rst. Also supply of LEDs - vccio or usbvdd? Change Rs if necessary change on vccio/usbvdd\nTest points?
 $EndSCHEMATC

Commit message: More changes on list to v0.2.
Parts:
- removed R3: 10k, symbol R
- added D6: ZENER, symbol ZENER
Connections:
- wire segments 121 -> 122
Other:
- note added: "Still TODO for v0.2:\nChange 3105 to 3108 for lower current operation?\n3.3v regulator from power sources to xbee pin 1\nSignaling from 3105 that it is not supplying current\nExternal/high voltage power terminal - traditional PV 6-12v\n Pull DRV off 4070 to pin for high current charging?\nJumpers for... what needs jumpers? Something must. \n Charge full indicator? Tx/Rx LEDs? USB vdd?\nMove PV co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"
- note removed: "Possible changes for v0.2:\nChange 3105 to 3108 for lower current operation?\nZener diode between usb_vdd and gnd.\n3.3v regulator from power sources to xbee pin 1\nSignaling from 3105 that it is not supplying current\nExternal/high voltage power terminal - traditional PV 6-12v\n Pull DRV off 4070 to pin for high current charging?\nJumpers for... what needs jumpers? Something must. \n Charge full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"
Changed lines of the file:
@@
 USB_VDD
 $Comp
-L GND #PWR01
+L GND #PWR4
 U 1 1 522EC0A5
 P 4250 7600
-F 0 "#PWR01" H 4250 7600 30  0001 C CNN
+F 0 "#PWR4" H 4250 7600 30  0001 C CNN
 F 1 "GND" H 4250 7530 30  0001 C CNN
 F 2 "" H 4250 7600 60  0000 C CNN
@@
 $EndComp
 $Comp
-L GND #PWR02
+L GND #PWR2
 U 1 1 522ECD60
 P 2350 5450
-F 0 "#PWR02" H 2350 5450 30  0001 C CNN
+F 0 "#PWR2" H 2350 5450 30  0001 C CNN
 F 1 "GND" H 2350 5380 30  0001 C CNN
 F 2 "" H 2350 5450 60  0000 C CNN
@@
 $EndComp
 $Comp
-L R R3
-U 1 1 522FE6E8
-P 3150 5200
-F 0 "R3" V 3230 5200 40  0000 C CNN
-F 1 "10k" V 3157 5201 40  0000 C CNN
-F 2 "" V 3080 5200 30  0000 C CNN
-F 3 "" H 3150 5200 30  0000 C CNN
-	1    3150 5200
-	1    0    0    -1
-$EndComp
-$Comp
 L C C9
 U 1 1 522FE8A3
@@
 $EndComp
 $Comp
-L GND #PWR03
+L GND #PWR1
 U 1 1 522FF942
 P 1450 7400
-F 0 "#PWR03" H 1450 7400 30  0001 C CNN
+F 0 "#PWR1" H 1450 7400 30  0001 C CNN
 F 1 "GND" H 1450 7330 30  0001 C CNN
 F 2 "" H 1450 7400 60  0000 C CNN
@@
 $EndComp
 $Comp
-L GND #PWR04
+L GND #PWR3
 U 1 1 52312207
 P 2800 3950
-F 0 "#PWR04" H 2800 3950 30  0001 C CNN
+F 0 "#PWR3" H 2800 3950 30  0001 C CNN
 F 1 "GND" H 2800 3880 30  0001 C CNN
 F 2 "" H 2800 3950 60  0000 C CNN
@@
 Zener reverse current between USB-VDD and GND? \nProbably should...
 $Comp
-L GND #PWR05
+L GND #PWR6
 U 1 1 52315DFC
 P 9200 3800
-F 0 "#PWR05" H 9200 3800 30  0001 C CNN
+F 0 "#PWR6" H 9200 3800 30  0001 C CNN
 F 1 "GND" H 9200 3730 30  0001 C CNN
 F 2 "" H 9200 3800 60  0000 C CNN
@@
 Connection ~ 4250 7350
 Wire Wire Line
-	3350 5850 3150 5850
+	3150 5850 3350 5850
 Connection ~ 4350 4650
 Wire Wire Line
-	3150 5850 3150 5450
-Wire Wire Line
-	3150 4950 3150 4550
+	3150 4850 3150 5850
 Wire Wire Line
 	2150 4550 4150 4550
@@
 	5600 4050 5850 4050
 Connection ~ 4150 4550
-Connection ~ 3150 4550
 Wire Wire Line
 	4150 4550 4150 4850
@@
 	2000 7050 2000 6300
 Wire Wire Line
-	1450 7050 2000 7050
+	1450 7050 3000 7050
 Wire Wire Line
 	9900 2150 10300 2150
@@
 	7800 1350 7900 1350
 $Comp
-L GND #PWR06
+L GND #PWR5
 U 1 1 5235B126
 P 5950 5350
-F 0 "#PWR06" H 5950 5350 30  0001 C CNN
+F 0 "#PWR5" H 5950 5350 30  0001 C CNN
 F 1 "GND" H 5950 5280 30  0001 C CNN
 F 2 "" H 5950 5350 60  0000 C CNN
@@
 NoConn ~ 5150 5450
 Text Notes 8650 700  0    60   ~ 0
-Possible changes for v0.2:\nChange 3105 to 3108 for lower current operation?\nZener diode between usb_vdd and gnd.\n3.3v regulator from power sources to xbee pin 1\nSignaling from 3105 that it is not supplying current\nExternal/high voltage power terminal - traditional PV 6-12v\n  Pull DRV off 4070 to pin for high current charging?\nJumpers for... what needs jumpers? Something must. \n  Charge full indicator? Tx/Rx LEDs? USB vdd?\nSwitch instead of diode isolation for USB/PV power selection? -NO!\nUSB Mirrored Insertion Footprint - !Impossible!\nMove battery holder up/change left smt header.\nMove PV connector pins.\nReexamine 10k pullup on #rst. Also supply of LEDs - vccio or usbvdd? Change Rs if necessary change on vccio/usbvdd\nTest points?
+Still TODO for v0.2:\nChange 3105 to 3108 for lower current operation?\n3.3v regulator from power sources to xbee pin 1\nSignaling from 3105 that it is not supplying current\nExternal/high voltage power terminal - traditional PV 6-12v\n  Pull DRV off 4070 to pin for high current charging?\nJumpers for... what needs jumpers? Something must. \n  Charge full indicator? Tx/Rx LEDs? USB vdd?\nMove PV connector pins.\nReexamine supply of LEDs - vccio or usbvdd? Change Rs if necessary change on vccio/usbvdd\nTest points?
+Connection ~ 3150 4850
+$Comp
+L ZENER D6
+U 1 1 5254E5F2
+P 3000 6050
+F 0 "D6" H 3000 6150 50  0000 C CNN
+F 1 "ZENER" H 3000 5950 40  0000 C CNN
+F 2 "" H 3000 6050 60  0000 C CNN
+F 3 "" H 3000 6050 60  0000 C CNN
+	1    3000 6050
+	0    -1   -1   0
+$EndComp
+Wire Wire Line
+	3000 7050 3000 6250
+Connection ~ 2000 7050
+Wire Wire Line
+	3000 5850 3000 4550
+Connection ~ 3000 4550
 $EndSCHEMATC

Commit message: Moving away from LTC310X DCDC converters.
Other:
- note added: "Still TODO for v0.2:\nChange 3105 to 3108 for lower current operation?\nIs a DC/DC converter really necessary? Could just try to pick an appropriate PV cell.\n3.3v regulator from power sources to xbee pin 1\nSignaling from 3105 that it is not supplying current\nExternal/high voltage power terminal - traditional PV 6-12v\n Pull DRV off 4070 to pin for high current charging?\nJumpers for... what ne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"
- note removed: "Still TODO for v0.2:\nChange 3105 to 3108 for lower current operation?\n3.3v regulator from power sources to xbee pin 1\nSignaling from 3105 that it is not supplying current\nExternal/high voltage power terminal - traditional PV 6-12v\n Pull DRV off 4070 to pin for high current charging?\nJumpers for... what needs jumpers? Something must. \n Charge full indicator? Tx/Rx LEDs? USB vdd?\nMove PV co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"
Changed lines of the file:
@@
 	1    0    0    -1
 $EndComp
-Text Notes 4650 2450 0    79   ~ 0
-Is this the best way to integrate \nUSB PWR and LTC3105 VOut??
 Text Notes 7050 2100 0    60   ~ 0
 ADJ -> Vcc \n= 4.2v Vout.\nADJ  -> NC\n=4.1v Vout.
@@
 NoConn ~ 5150 5450
 Text Notes 8650 700  0    60   ~ 0
-Still TODO for v0.2:\nChange 3105 to 3108 for lower current operation?\n3.3v regulator from power sources to xbee pin 1\nSignaling from 3105 that it is not supplying current\nExternal/high voltage power terminal - traditional PV 6-12v\n  Pull DRV off 4070 to pin for high current charging?\nJumpers for... what needs jumpers? Something must. \n  Charge full indicator? Tx/Rx LEDs? USB vdd?\nMove PV connector pins.\nReexamine supply of LEDs - vccio or usbvdd? Change Rs if necessary change on vccio/usbvdd\nTest points?
+Still TODO for v0.2:\nChange 3105 to 3108 for lower current operation?\nIs a DC/DC converter really necessary? Could just try to pick an appropriate PV cell.\n3.3v regulator from power sources to xbee pin 1\nSignaling from 3105 that it is not supplying current\nExternal/high voltage power terminal - traditional PV 6-12v\n  Pull DRV off 4070 to pin for high current charging?\nJumpers for... what needs jumpers? Something must. \n  Charge full indicator? Tx/Rx LEDs? USB vdd?\nMove PV connector pins.\nReexamine supply of LEDs - vccio or usbvdd? Change Rs if necessary change on vccio/usbvdd\nTest points?
 Connection ~ 3150 4850
 $Comp
@@
 	3000 5850 3000 4550
 Connection ~ 3000 4550
+Text Notes 4650 2450 0    79   ~ 0
+Is this the best way to integrate \nUSB PWR and LTC3105 VOut??
 $EndSCHEMATC

Commit message: Almost everything on the TODO is done. Layout done.
Parts:
- removed C2: 1uF, symbol C
- removed C6: 4.7uF, symbol C
- removed C8: 10uF, symbol C
- removed D3, D4: DIODESCH, symbol DIODESCH
- removed L1: 10uH, symbol INDUCTOR
- removed R4: 3.3M, symbol R
- removed R5: 1M, symbol R
- removed U3: LTC3105-MSOP12, symbol LTC3105-MSOP12
- added D3, D4, D7: DIODE-NC, symbol DIODE-NC
- added R3: 22R, symbol R
- added U2: AP7313-3.3VREGULATOR, symbol AP7313-3.3VREGULATOR
- R6: value 33R -> 22R
Connections:
- wire segments 122 -> 98
Other:
- note added: "D3/D4 Fw Drop Approx. 0.7V\nAssume 5V for PC"
- note added: "R6 chosen to limit shunt current to 50mA.\n(4.3v-3.2v)/22=50mA max charge current.\n(4.3v-3.2v)^2/33=55mW PwrDiss\n(4.3v-4.1v)/33=3.03mA max shunt current.\n"
- note added: "Still TODO for v0.2:\nJumpers for... what needs jumpers? Something must. \n Charge full indicator? Tx/Rx LEDs? USB vdd?\nTest points?"
- note removed: "D3/D4 Fw Drop <.2V"
- note removed: "Is this the best way to integrate \nUSB PWR and LTC3105 VOut??"
- note removed: "PGood or LDO can be used to signal uController \nthat PVCell is not charging... not used currently.\nOpen drain so use a pull-up.\nSuggest PB4/Pin7 as PCINT or just I/O on MT."
- note removed: "R6 to be chosen to \nlimit shunt current to 50mA.\n(4.8v-3.2v)/33=48mA max charge current.\n(4.8v-3.2v)^2/33=77.5mW PwrDiss\n(4.8v-4.1v)/33=21.2mA max shunt current.\nNeed to double check these numbers."
- note removed: "Still TODO for v0.2:\nChange 3105 to 3108 for lower current operation?\nIs a DC/DC converter really necessary? Could just try to pick an appropriate PV cell.\n3.3v regulator from power sources to xbee pin 1\nSignaling from 3105 that it is not supplying current\nExternal/high voltage power terminal - traditional PV 6-12v\n Pull DRV off 4070 to pin for high current charging?\nJumpers for... what ne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"
- note removed: "VOut = 1.004v(R4/R5+1) = LTC4070Vcc + diode drop on D4.\nShould be in MOhm range.\n1.004*(3.3+1) = 4.3172V\nLDO = 1.004v(Vdiv between LDO/FBLDO+1) - Not used.\n"
- moved on the sheet: C1, P2, R6

Commit message: Added mounting holes, some SMT jumpers and a voltage divider. Extended board for mounts by 3.5mm.
Parts:
- added JP1, JP2, JP3: JUMPER, symbol JUMPER
- added R4, R5: 22k, symbol R
Connections:
- net labels added: _MT_PB4, _MT_PF7
- wire segments 98 -> 116
- no-connect marks 47 -> 45
Changed lines of the file:
@@
 $EndComp
 NoConn ~ 9500 5200
-NoConn ~ 9500 5100
 NoConn ~ 9500 5000
 NoConn ~ 9500 4900
@@
 NoConn ~ 5950 4600
 NoConn ~ 5950 4800
-NoConn ~ 5950 4900
 NoConn ~ 5950 5000
 NoConn ~ 5950 5100
@@
 Connection ~ 6750 3600
 NoConn ~ 6900 2700
+Text GLabel 8950 2900 3    60   Input ~ 0
+_MT_PB4
+Wire Wire Line
+	8950 2900 8950 2750
+Connection ~ 8950 2750
+Text GLabel 4750 4150 0    60   Input ~ 0
+_MT_PB4
+Wire Wire Line
+	5950 4900 5850 4900
+Wire Wire Line
+	5850 4900 5850 4650
+$Comp
+L JUMPER JP1
+U 1 1 525BDBD8
+P 5100 4450
+F 0 "JP1" H 5100 4600 60  0000 C CNN
+F 1 "JUMPER" H 5100 4370 40  0000 C CNN
+F 2 "" H 5100 4450 60  0000 C CNN
+F 3 "" H 5100 4450 60  0000 C CNN
+	1    5100 4450
+	1    0    0    -1
+$EndComp
+Wire Wire Line
+	5400 4450 5400 4650
+Wire Wire Line
+	5400 4650 5850 4650
+Wire Wire Line
+	4750 4150 4800 4150
+Wire Wire Line
+	4800 4150 4800 4450
+$Comp
+L JUMPER JP2
+U 1 1 525BDD98
+P 8950 900
+F 0 "JP2" H 8950 1050 60  0000 C CNN
+F 1 "JUMPER" H 8950 820 40  0000 C CNN
+F 2 "" H 8950 900 60  0000 C CNN
+F 3 "" H 8950 900 60  0000 C CNN
+	1    8950 900
+	1    0    0    -1
+$EndComp
+Wire Wire Line
+	7100 1350 7100 900
+Connection ~ 7100 1350
+$Comp
+L R R4
+U 1 1 525BDECB
+P 9400 1150
+F 0 "R4" V 9480 1150 40  0000 C CNN
+F 1 "22k" V 9407 1151 40  0000 C CNN
+F 2 "" V 9330 1150 30  0000 C CNN
+F 3 "" H 9400 1150 30  0000 C CNN
+	1    9400 1150
+	-1   0    0    1
+$EndComp
+$Comp
+L R R5
+U 1 1 525BDF6F
+P 9750 1200
+F 0 "R5" V 9830 1200 40  0000 C CNN
+F 1 "22k" V 9757 1201 40  0000 C CNN
+F 2 "" V 9680 1200 30  0000 C CNN
+F 3 "" H 9750 1200 30  0000 C CNN
+	1    9750 1200
+	1    0    0    -1
+$EndComp
+Wire Wire Line
+	9400 1550 9600 1550
+Wire Wire Line
+	9600 1550 9600 900
+Wire Wire Line
+	9600 900  10050 900
+Wire Wire Line
+	9750 900  9750 950
+$Comp
+L GND #PWR06
+U 1 1 525BE0CC
+P 9750 1650
+F 0 "#PWR06" H 9750 1650 30  0001 C CNN
+F 1 "GND" H 9750 1580 30  0001 C CNN
+F 2 "" H 9750 1650 60  0000 C CNN
+F 3 "" H 9750 1650 60  0000 C CNN
+	1    9750 1650
+	1    0    0    -1
+$EndComp
+Wire Wire Line
+	9750 1450 9750 1650
+Text GLabel 10050 900  2    60   Input ~ 0
+_MT_PF7
+Connection ~ 9750 900
+Text GLabel 10400 5100 2    60   Input ~ 0
+_MT_PF7
+Wire Wire Line
+	9250 900  9400 900
+Wire Wire Line
+	9400 1400 9400 1550
+$Comp
+L JUMPER JP3
+U 1 1 525BE6B9
+P 10000 5100
+F 0 "JP3" H 10000 5250 60  0000 C CNN
+F 1 "JUMPER" H 10000 5020 40  0000 C CNN
+F 2 "" H 10000 5100 60  0000 C CNN
+F 3 "" H 10000 5100 60  0000 C CNN
+	1    10000 5100
+	1    0    0    -1
+$EndComp
+Wire Wire Line
+	10300 5100 10400 5100
+Wire Wire Line
+	9700 5100 9500 5100
+Wire Wire Line
+	7100 900  8650 900
 $EndSCHEMATC

Commit message: Change all the things\!
Connections:
- net labels added: _MT_PF2, _MT_PF3
- net labels removed: _MT_PB4, _MT_PF7
- wire segments 116 -> 113
Other:
- moved on the sheet: JP1, JP3
Changed lines of the file:
@@
 NoConn ~ 9500 4800
 NoConn ~ 9500 4700
-NoConn ~ 9500 4600
-NoConn ~ 9500 4500
 NoConn ~ 9500 4400
 NoConn ~ 9500 4300
@@
 NoConn ~ 6900 2700
 Text GLabel 8950 2900 3    60   Input ~ 0
-_MT_PB4
+_MT_PF2
 Wire Wire Line
 	8950 2900 8950 2750
 Connection ~ 8950 2750
-Text GLabel 4750 4150 0    60   Input ~ 0
-_MT_PB4
-Wire Wire Line
-	5950 4900 5850 4900
-Wire Wire Line
-	5850 4900 5850 4650
+Text GLabel 10400 4300 2    60   Input ~ 0
+_MT_PF2
 $Comp
 L JUMPER JP1
 U 1 1 525BDBD8
-P 5100 4450
-F 0 "JP1" H 5100 4600 60  0000 C CNN
-F 1 "JUMPER" H 5100 4370 40  0000 C CNN
-F 2 "" H 5100 4450 60  0000 C CNN
-F 3 "" H 5100 4450 60  0000 C CNN
-	1    5100 4450
-	1    0    0    -1
-$EndComp
-Wire Wire Line
-	5400 4450 5400 4650
-Wire Wire Line
-	5400 4650 5850 4650
-Wire Wire Line
-	4750 4150 4800 4150
-Wire Wire Line
-	4800 4150 4800 4450
+P 10000 4300
+F 0 "JP1" H 10000 4450 60  0000 C CNN
+F 1 "JUMPER" H 10000 4220 40  0000 C CNN
+F 2 "" H 10000 4300 60  0000 C CNN
+F 3 "" H 10000 4300 60  0000 C CNN
+	1    10000 4300
+	1    0    0    -1
+$EndComp
 $Comp
 L JUMPER JP2
@@
 	9750 1450 9750 1650
 Text GLabel 10050 900  2    60   Input ~ 0
-_MT_PF7
+_MT_PF3
 Connection ~ 9750 900
-Text GLabel 10400 5100 2    60   Input ~ 0
-_MT_PF7
+Text GLabel 10400 4600 2    60   Input ~ 0
+_MT_PF3
 Wire Wire Line
 	9250 900  9400 900
@@
 L JUMPER JP3
 U 1 1 525BE6B9
-P 10000 5100
-F 0 "JP3" H 10000 5250 60  0000 C CNN
-F 1 "JUMPER" H 10000 5020 40  0000 C CNN
-F 2 "" H 10000 5100 60  0000 C CNN
-F 3 "" H 10000 5100 60  0000 C CNN
-	1    10000 5100
-	1    0    0    -1
-$EndComp
-Wire Wire Line
-	10300 5100 10400 5100
-Wire Wire Line
-	9700 5100 9500 5100
+P 10000 4600
+F 0 "JP3" H 10000 4750 60  0000 C CNN
+F 1 "JUMPER" H 10000 4520 40  0000 C CNN
+F 2 "" H 10000 4600 60  0000 C CNN
+F 3 "" H 10000 4600 60  0000 C CNN
+	1    10000 4600
+	1    0    0    -1
+$EndComp
+Wire Wire Line
+	10300 4600 10400 4600
+Wire Wire Line
+	9700 4600 9500 4600
 Wire Wire Line
 	7100 900  8650 900
+NoConn ~ 5950 4900
+NoConn ~ 9500 5100
+Wire Wire Line
+	10400 4300 10300 4300
+Wire Wire Line
+	9700 4300 9700 4500
+Wire Wire Line
+	9700 4500 9500 4500
 $EndSCHEMATC

Commit message: Mark for changes for v0.3.
Other:
- note added: "Optional Charge \nFull Indicator...\nOtherwise NC HBO\n...Active High!\nSeems this doesn't light when MT is inserted, \nmaybe fixed by changing R6, D3 or both."
- note added: "Still TODO for v0.3:\nBetter values for current limiting Rs to charging circuitry.\nC1 lower value, higher voltage rating.\nPads for higher current charging/DRV on 4070.\nFiducials.\nReconsider changing back to shottkey diodes for charging circuitry.\nJumpers for... what needs jumpers? Something must. \n Charge full indicator? Tx/Rx LEDs? USB vdd?\nTest points?\n"
- note removed: "Optional Charge \nFull Indicator...\nOtherwise NC HBO\n...Active High!"
- note removed: "Still TODO for v0.2:\nJumpers for... what needs jumpers? Something must. \n Charge full indicator? Tx/Rx LEDs? USB vdd?\nTest points?"
- note removed: "Zener reverse current between USB-VDD and GND? \nProbably should..."
Changed lines of the file:
@@
 Text GLabel 3300 1850 0    60   Input ~ 0
 USB_VDD
-Text Notes 1550 7250 0    60   ~ 0
-Zener reverse current between USB-VDD and GND? \nProbably should...
 $Comp
 L GND #PWR04
@@
 	1    0    0    -1
 $EndComp
-Text Notes 9400 3100 0    60   ~ 0
-Optional Charge \nFull Indicator...\nOtherwise NC HBO\n...Active High!
+Text Notes 9150 3550 0    60   ~ 0
+Optional Charge \nFull Indicator...\nOtherwise NC HBO\n...Active High!\nSeems this doesn't light when MT is inserted, \nmaybe fixed by changing R6, D3 or both.
 Text Notes 2750 1100 0    60   ~ 0
 R6 chosen to limit shunt current to 50mA.\n(4.3v-3.2v)/22=50mA max charge current.\n(4.3v-3.2v)^2/33=55mW PwrDiss\n(4.3v-4.1v)/33=3.03mA max shunt current.\n
@@
 NoConn ~ 5150 5550
 NoConn ~ 5150 5450
-Text Notes 650  3300 0    60   ~ 0
-Still TODO for v0.2:\nJumpers for... what needs jumpers? Something must. \n  Charge full indicator? Tx/Rx LEDs? USB vdd?\nTest points?
+Text Notes 850  3950 0    60   ~ 0
+Still TODO for v0.3:\nBetter values for current limiting Rs to charging circuitry.\nC1 lower value, higher voltage rating.\nPads for higher current charging/DRV on 4070.\nFiducials.\nReconsider changing back to shottkey diodes for charging circuitry.\nJumpers for... what needs jumpers? Something must. \n  Charge full indicator? Tx/Rx LEDs? USB vdd?\nTest points?\n
 Connection ~ 3150 4850
 $Comp
