File: Hardware/MeshUSB.sch (KiCad schematic (older format))
At the start: 37 parts, among them P1 USB_4, P2 PVCell, Q1 MOS_P, U1 XBEE, U2 AP7313-3.3VREGULATOR, U4 FT231X-SSOP, U5 LTC4070

Commit message: Begin Layout. Still some schematic additions required.
Parts:
- renumbered F1 to Fi1, F2 to Fi2, F3 to Fi3
Changed lines of the file:
@@
 	4850 2000 10350 2000
 $Comp
-L CONN_1 F1
+L CONN_1 Fi1
 U 1 1 53044226
 P 10100 5700
-F 0 "F1" H 10180 5700 40  0000 L CNN
+F 0 "Fi1" H 10180 5700 40  0000 L CNN
 F 1 "CONN_1" H 10100 5755 30  0001 C CNN
 F 2 "" H 10100 5700 60  0000 C CNN
@@
 $EndComp
 $Comp
-L CONN_1 F2
+L CONN_1 Fi2
 U 1 1 5304423A
 P 10100 5800
-F 0 "F2" H 10180 5800 40  0000 L CNN
+F 0 "Fi2" H 10180 5800 40  0000 L CNN
 F 1 "CONN_1" H 10100 5855 30  0001 C CNN
 F 2 "" H 10100 5800 60  0000 C CNN
@@
 $EndComp
 $Comp
-L CONN_1 F3
+L CONN_1 Fi3
 U 1 1 5304424E
 P 10100 5900
-F 0 "F3" H 10180 5900 40  0000 L CNN
+F 0 "Fi3" H 10180 5900 40  0000 L CNN
 F 1 "CONN_1" H 10100 5955 30  0001 C CNN
 F 2 "" H 10100 5900 60  0000 C CNN

Commit message: Further changes. Still looking for appropriate diode and PMOS packages.
Parts:
- added JP4: JUMPER, symbol JUMPER
- R4: value 22k -> 33k
- R5: value 22k -> 20k
Connections:
- net labels added: _MT_PE4
- wire segments 109 -> 112
- no-connect marks 47 -> 46
Changed lines of the file:
@@
 	-1   0    0    1
 $EndComp
-NoConn ~ 9500 5200
 NoConn ~ 9500 5000
 NoConn ~ 9500 4900
@@
 P 9400 1150
 F 0 "R4" V 9480 1150 40  0000 C CNN
-F 1 "22k" V 9407 1151 40  0000 C CNN
+F 1 "33k" V 9407 1151 40  0000 C CNN
 F 2 "" V 9330 1150 30  0000 C CNN
 F 3 "" H 9400 1150 30  0000 C CNN
@@
 P 9750 1200
 F 0 "R5" V 9830 1200 40  0000 C CNN
-F 1 "22k" V 9757 1201 40  0000 C CNN
+F 1 "20k" V 9757 1201 40  0000 C CNN
 F 2 "" V 9680 1200 30  0000 C CNN
 F 3 "" H 9750 1200 30  0000 C CNN
@@
 Wire Wire Line
 	9750 900  9750 950
-$Comp
-L GND #PWR06
-U 1 1 525BE0CC
-P 9750 1650
-F 0 "#PWR06" H 9750 1650 30  0001 C CNN
-F 1 "GND" H 9750 1580 30  0001 C CNN
-F 2 "" H 9750 1650 60  0000 C CNN
-F 3 "" H 9750 1650 60  0000 C CNN
-	1    9750 1650
-	1    0    0    -1
-$EndComp
 Wire Wire Line
 	9750 1450 9750 1650
@@
 	6000 2700 6000 3050
 Connection ~ 6000 3050
+$Comp
+L JUMPER JP4
+U 1 1 53057C45
+P 10000 5200
+F 0 "JP4" H 10000 5350 60  0000 C CNN
+F 1 "JUMPER" H 10000 5120 40  0000 C CNN
+F 2 "" H 10000 5200 60  0000 C CNN
+F 3 "" H 10000 5200 60  0000 C CNN
+	1    10000 5200
+	1    0    0    -1
+$EndComp
+Text GLabel 10400 5200 2    60   Input ~ 0
+_MT_PE4
+Text GLabel 10050 1650 2    60   Input ~ 0
+_MT_PE4
+Wire Wire Line
+	9750 1650 10050 1650
+Wire Wire Line
+	10400 5200 10300 5200
+Wire Wire Line
+	9700 5200 9500 5200
 $EndSCHEMATC

Commit message: Schematic notes and library updates.
Parts:
- removed JP2: JUMPER, symbol JUMPER
- added JP?: CONN_TH_JMPR_DEFAULTCLOSED, symbol CONN_TH_JMPR_DEFAULTCLOSED
- added P?: CONN_2, symbol CONN_2
- added U?: DUALPMOS-ZXMD63P02X, symbol DUALPMOS-ZXMD63P02X
Connections:
- wire segments 112 -> 114
Other:
- note added: "Approx. 6V max. without further current limiting. \nDiode forward current is 200mA."
- note added: "Exposed pins for charging... User must be careful!\nDo these as JST 2mm?"
- note added: "RDS on might not be sufficiently low for shunt current...\nFind a better choice."
- note added: "Still TODO for v0.3:\nFind DRV/low batter cutoff dual PMOS package or descrets.\nJumpers for... what needs jumpers? Something must. \n Cutoff battery charging. Charge full indicator? Tx/Rx LEDs? USB vdd?\nTest points?\n"
- note added: "This is for disabling \nsoft reset ~DTR.\nMake as two .254mm THs \nconnected by default."
- note added: "V.Div. Gives limited range. Get numbers from spreadsheet."
- note removed: "Still TODO for v0.3:\nC1 lower value, higher voltage rating.\nPads for higher current charging/DRV on 4070.\nJumpers for... what needs jumpers? Something must. \n Cutoff battery charging. Charge full indicator? Tx/Rx LEDs? USB vdd?\nTest points?\nJumper/switch for enable/disable ~DTR reset.\n"
- moved on the sheet: C9

Commit message: Higher current charging. Some datasheets.
Parts:
- added Q?: MOS_P-INFINEON-BSS83P, symbol MOS_P-INFINEON-BSS83P
Connections:
- wire segments 114 -> 117
- no-connect marks 46 -> 45
Changed lines of the file:
@@
 Text Notes 3650 2350 0    60   ~ 0
 Fw Drop Approx. 0.5V @ 100mA
-NoConn ~ 8550 3000
 $Comp
 L MOS_P-INFINEON-BSS83P Q1
@@
 $EndComp
 NoConn ~ 6900 2700
-Text GLabel 8950 2900 3    60   Input ~ 0
+Text GLabel 9150 2650 1    60   Input ~ 0
 _MT_PF2
 Text GLabel 10400 4300 2    60   Input ~ 0
@@
 Connection ~ 6750 3600
 Wire Wire Line
-	8950 2900 8950 2750
-Connection ~ 8950 2750
-Wire Wire Line
 	7100 1350 7100 900
 Connection ~ 7100 1350
@@
 	1    0    0    -1
 $EndComp
+$Comp
+L MOS_P-INFINEON-BSS83P Q?
+U 1 1 53080F7D
+P 8800 3000
+F 0 "Q?" H 8800 3190 60  0000 R CNN
+F 1 "MOS_P-INFINEON-BSS83P" H 8800 2820 60  0001 R CNN
+F 2 "" H 8800 3000 60  0000 C CNN
+F 3 "" H 8800 3000 60  0000 C CNN
+	1    8800 3000
+	1    0    0    1
+$EndComp
+Wire Wire Line
+	8550 3000 8600 3000
+Connection ~ 8900 2000
+Wire Wire Line
+	8900 3200 8900 3600
+Connection ~ 8900 3600
+Wire Wire Line
+	9150 2650 9150 2750
+Connection ~ 9150 2750
+Wire Wire Line
+	8900 2000 8900 2800
 $EndSCHEMATC

Commit message: Almost to layout. Charging slightly modified, confirming BOM.
Parts:
- removed D30: BAT54C, symbol BAT54C
- removed U?: DUALPMOS-ZXMD63P02X, symbol DUALPMOS-ZXMD63P02X
- added D30: DUAL_SHOTTKEY_PACKAGE, symbol DUAL_SHOTTKEY_PACKAGE
- R30: value 10R -> 16R
- gave numbers to parts that had none: 3
Other:
- note added: "Approx. 6V max. without further current limiting. \nDiode forward current is 500mA."
- note added: "Charging max values\ncharge I - 125mA=1C battery\nPwrDiss - 2W - depends on R30\nshunt I - 50 mA\n"
- note added: "Fw Drop Approx. \n0.2V @ 100mA\n0.3V @ 500mA\n"
- note added: "Still TODO for v0.3:\nJumpers for... what needs jumpers? Something must. \n Cutoff battery charging. Charge full indicator? Tx/Rx LEDs? USB vdd?\nTest points?\n"
- note removed: "Approx. 6V max. without further current limiting. \nDiode forward current is 200mA."
- note removed: "Charging max values\ncharge I - 125mA=1C battery\nPwrDiss - 200mW (?) - depends on R3\nshunt I - 50 mA\n"
- note removed: "Fw Drop Approx. 0.5V @ 100mA"
- note removed: "RDS on might not be sufficiently low for shunt current...\nFind a better choice."
- note removed: "Still TODO for v0.3:\nFind DRV/low batter cutoff dual PMOS package or descrets.\nJumpers for... what needs jumpers? Something must. \n Cutoff battery charging. Charge full indicator? Tx/Rx LEDs? USB vdd?\nTest points?\n"
Changed lines of the file:
@@
 Text GLabel 5950 1350 0    60   Input ~ 0
 BAT+
-Text Notes 3650 2350 0    60   ~ 0
-Fw Drop Approx. 0.5V @ 100mA
+Text Notes 4400 2350 0    60   ~ 0
+Fw Drop Approx. \n0.2V @ 100mA\n0.3V @ 500mA\n
 $Comp
 L MOS_P-INFINEON-BSS83P Q1
@@
 NoConn ~ 5150 5450
 Text Notes 850  3950 0    60   ~ 0
-Still TODO for v0.3:\nFind DRV/low batter cutoff dual PMOS package or descrets.\nJumpers for... what needs jumpers? Something must. \n  Cutoff battery charging. Charge full indicator? Tx/Rx LEDs? USB vdd?\nTest points?\n
+Still TODO for v0.3:\nJumpers for... what needs jumpers? Something must. \n  Cutoff battery charging. Charge full indicator? Tx/Rx LEDs? USB vdd?\nTest points?\n
 $Comp
 L ZENER D6
@@
 P 4600 2000
 F 0 "R30" V 4680 2000 40  0000 C CNN
-F 1 "10R" V 4607 2001 40  0000 C CNN
+F 1 "16R" V 4607 2001 40  0000 C CNN
 F 2 "" V 4530 2000 30  0000 C CNN
 F 3 "" H 4600 2000 30  0000 C CNN
@@
 NoConn ~ 9500 5100
 Text Notes 3650 1600 0    60   ~ 0
-Charging max values\ncharge I - 125mA=1C battery\nPwrDiss - 200mW (?) - depends on R3\nshunt I - 50 mA\n
+Charging max values\ncharge I - 125mA=1C battery\nPwrDiss - 2W - depends on R30\nshunt I - 50 mA\n
 NoConn ~ 7250 2600
-$Comp
-L BAT54C D30
-U 1 1 530432F5
-P 3900 2000
-F 0 "D30" H 3750 2250 40  0000 C CNN
-F 1 "BAT54C" H 4000 1750 40  0000 C CNN
-F 2 "" H 3800 1900 60  0000 C CNN
-F 3 "" H 3800 1900 60  0000 C CNN
-	1    3900 2000
-	1    0    0    -1
-$EndComp
 $Comp
 L CONN_1 Fi1
@@
 _MT_PE4
 $Comp
-L DUALPMOS-ZXMD63P02X U?
-U 1 1 5307F349
-P 1600 1050
-F 0 "U?" H 1500 1350 60  0000 C CNN
-F 1 "DUALPMOS-ZXMD63P02X" H 1650 750 60  0000 C CNN
-F 2 "" H 1600 1050 60  0000 C CNN
-F 3 "" H 1600 1050 60  0000 C CNN
-	1    1600 1050
-	1    0    0    -1
-$EndComp
-$Comp
-L CONN_2 P?
+L CONN_2 P30
 U 1 1 5307F372
 P 10800 2600
-F 0 "P?" V 10750 2600 40  0000 C CNN
+F 0 "P30" V 10750 2600 40  0000 C CNN
 F 1 "CONN_2" V 10850 2600 40  0000 C CNN
 F 2 "" H 10800 2600 60  0000 C CNN
@@
 V.Div. Gives limited range. Get numbers from spreadsheet.
 Text Notes 650  2400 0    60   ~ 0
-Approx. 6V max. without further current limiting. \nDiode forward current is 200mA.
-Text Notes 1200 700  0    60   ~ 0
-RDS on might not be sufficiently low for shunt current...\nFind a better choice.
+Approx. 6V max. without further current limiting. \nDiode forward current is 500mA.
 Text Notes 5000 4600 0    39   ~ 0
 This is for disabling \nsoft reset ~DTR.\nMake as two .254mm THs \nconnected by default.
@@
 	5850 4400 5950 4400
 $Comp
-L CONN_TH_JMPR_DEFAULTCLOSED JP?
+L CONN_TH_JMPR_DEFAULTCLOSED JP2
 U 1 1 5308067F
 P 5500 4700
-F 0 "JP?" H 5450 4600 40  0000 L CNN
+F 0 "JP2" H 5450 4600 40  0000 L CNN
 F 1 "CONN_TH_JMPR_DEFAULTCLOSED" H 5500 4800 30  0001 C CNN
 F 2 "" H 5500 4700 60  0000 C CNN
@@
 $EndComp
 $Comp
-L MOS_P-INFINEON-BSS83P Q?
+L MOS_P-INFINEON-BSS83P Q2
 U 1 1 53080F7D
 P 8800 3000
-F 0 "Q?" H 8800 3190 60  0000 R CNN
+F 0 "Q2" H 8800 3190 60  0000 R CNN
 F 1 "MOS_P-INFINEON-BSS83P" H 8800 2820 60  0001 R CNN
 F 2 "" H 8800 3000 60  0000 C CNN
@@
 Wire Wire Line
 	8900 2000 8900 2800
+$Comp
+L DUAL_SHOTTKEY_PACKAGE D30
+U 1 1 530A8D87
+P 3900 2000
+F 0 "D30" H 3750 2250 40  0000 C CNN
+F 1 "DUAL_SHOTTKEY_PACKAGE" H 4000 1750 40  0000 C CNN
+F 2 "" H 3800 1900 60  0000 C CNN
+F 3 "" H 3800 1900 60  0000 C CNN
+	1    3900 2000
+	1    0    0    -1
+$EndComp
 $EndSCHEMATC

Commit message: Layoutsplosion.
Parts:
- P30: value CONN_2 -> JST_2
Changed lines of the file:
@@
 P 10800 2600
 F 0 "P30" V 10750 2600 40  0000 C CNN
-F 1 "CONN_2" V 10850 2600 40  0000 C CNN
+F 1 "JST_2" V 10850 2600 40  0000 C CNN
 F 2 "" H 10800 2600 60  0000 C CNN
 F 3 "" H 10800 2600 60  0000 C CNN
 	1    10800 2600
-	1    0    0    -1
+	1    0    0    1
 $EndComp
 Text Notes 11050 2500 0    60   ~ 0

Commit message: Layout positions nearly finalized.
Other:
- note added: "Approx. 6V max. without further current limiting. \nDiode forward current max. is 500mA."
- note removed: "Approx. 6V max. without further current limiting. \nDiode forward current is 500mA."
Changed lines of the file:
@@
 V.Div. Gives limited range. Get numbers from spreadsheet.
 Text Notes 650  2400 0    60   ~ 0
-Approx. 6V max. without further current limiting. \nDiode forward current is 500mA.
+Approx. 6V max. without further current limiting. \nDiode forward current max. is 500mA.
 Text Notes 5000 4600 0    39   ~ 0
 This is for disabling \nsoft reset ~DTR.\nMake as two .254mm THs \nconnected by default.

Commit message: Further placements, silks, refs. Next:Double check all pins and packages.
Parts:
- R10, R8, R9: value 270 -> 270R
Changed lines of the file:
@@
 Sheet 1 1
 Title "MeshUSB by Robert Powers"
-Date "10 Sep 2013"
-Rev "v0.1"
-Comp "MeshAge"
+Date "24 Feb 2014"
+Rev "v0.3"
+Comp "M9Design.co"
 Comment1 ""
 Comment2 ""
@@
 P 5950 5950
 F 0 "R8" V 6030 5950 40  0000 C CNN
-F 1 "270" V 5957 5951 40  0000 C CNN
+F 1 "270R" V 5957 5951 40  0000 C CNN
 F 2 "" V 5880 5950 30  0000 C CNN
 F 3 "" H 5950 5950 30  0000 C CNN
@@
 P 6300 6050
 F 0 "R9" V 6380 6050 40  0000 C CNN
-F 1 "270" V 6307 6051 40  0000 C CNN
+F 1 "270R" V 6307 6051 40  0000 C CNN
 F 2 "" V 6230 6050 30  0000 C CNN
 F 3 "" H 6300 6050 30  0000 C CNN
@@
 P 9900 2400
 F 0 "R10" V 9980 2400 40  0000 C CNN
-F 1 "270" V 9907 2401 40  0000 C CNN
+F 1 "270R" V 9907 2401 40  0000 C CNN
 F 2 "" V 9830 2400 30  0000 C CNN
 F 3 "" H 9900 2400 30  0000 C CNN
