File: Hardware/MeshUSB.kicad_pcb (KiCad board)
At the start: 2 copper layers, 30.2 x 44.3 mm, 49 parts, among them P1 USB_4, P2 PVCell, P30 JST_2, P31 CONN_1, Q1 MOS_P, Q2 MOS_P-INFINEON-BSS83P, U1 XBEE, U2 AP7313-3.3VREGULATOR, U4 FT231X-SSOP, U5 LTC4070

Commit message: V0.3 production files.
Parts:
- H1: footprint _MUSB-FEMALE-HEADER-NPPN101BFLD-RC-Pin1Right -> _MUSB_:_MUSB-FEMALE-HEADER-NPPN101BFLD-RC-Pin1Right
- H2: footprint _MUSB-FEMALE-HEADER-NPPN101BFLC-RC-Pin1Left -> _MUSB_:_MUSB-FEMALE-HEADER-NPPN101BFLC-RC-Pin1Left
Changed lines of the file:
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@@
       (net 50 USB_VDD))
-  )
-  (module _MUSB-FEMALE-HEADER-NPPN101BFLD-RC-Pin1Right locked (layer F.Cu)
-    (at 137.5 114.004 180)
-    (attr smd)
-    (fp_text reference H1 (at 0 -11.47 180) (layer F.SilkS) hide
-      (effects (font (size 1 1) (thickness 0.15)))
-    )
-    (fp_text value XBeeLeftPins (at 0 11.57 180) (layer F.SilkS) hide
-      (effects (font (size 1 1) (thickness 0.15)))
-    )
-    (fp_line (start -1.2 8) (end 1.2 8) (layer F.SilkS) (width 0.15))
-    (fp_line (start 1.2 -10.25) (end 1.2 10.25) (layer F.SilkS) (width 0.15))
-    (fp_line (start 1.2 10.25) (end -1.2 10.25) (layer F.SilkS) (width 0.15))
-    (fp_line (start -1.2 10.25) (end -1.2 -10.25) (layer F.SilkS) (width 0.15))
-    (fp_line (start -1.2 -10.25) (end 1.2 -10.25) (layer F.SilkS) (width 0.15))
-    (pad 1 smd rect (at 2.54 9 180) (size 2.29 0.89) (layers F.Cu F.Paste F.Mask)
-      (net 6 BAT+))
-    (pad 2 smd rect (at -2.54 7 180) (size 2.29 0.89) (layers F.Cu F.Paste F.Mask)
-      (net 16 "Net-(H1-Pad2)"))
-    (pad 3 smd rect (at 2.54 5 180) (size 2.29 0.89) (layers F.Cu F.Paste F.Mask)
-      (net 17 "Net-(H1-Pad3)"))
-    (pad 4 smd rect (at -2.54 3 180) (size 2.29 0.89) (layers F.Cu F.Paste F.Mask)
-      (net 18 "Net-(H1-Pad4)"))
-    (pad 5 smd rect (at 2.54 1 180) (size 2.29 0.89) (layers F.Cu F.Paste F.Mask)
-      (net 19 "Net-(H1-Pad5)"))
-    (pad 6 smd rect (at -2.54 -1 180) (size 2.29 0.89) (layers F.Cu F.Paste F.Mask)
-      (net 20 "Net-(H1-Pad6)"))
-    (pad 7 smd rect (at 2.54 -3 180) (size 2.29 0.89) (layers F.Cu F.Paste F.Mask)
-      (net 21 "Net-(H1-Pad7)"))
-    (pad 8 smd rect (at -2.54 -5 180) (size 2.29 0.89) (layers F.Cu F.Paste F.Mask)
-      (net 22 "Net-(H1-Pad8)"))
-    (pad 9 smd rect (at 2.54 -7 180) (size 2.29 0.89) (layers F.Cu F.Paste F.Mask)
-      (net 23 "Net-(H1-Pad9)"))
-    (pad 10 smd rect (at -2.54 -9 180) (size 2.29 0.89) (layers F.Cu F.Paste F.Mask)
-      (net 7 GND))
-  )
-  (module _MUSB-FEMALE-HEADER-NPPN101BFLC-RC-Pin1Left locked (layer F.Cu)
-    (at 159.502 114.004)
-    (attr smd)
-    (fp_text reference H2 (at 0 -11.47) (layer F.SilkS) hide
-      (effects (font (size 1 1) (thickness 0.15)))
-    )
-    (fp_text value XBeeRightPins (at 0 11.57) (layer F.SilkS) hide
-      (effects (font (size 1 1) (thickness 0.15)))
-    )
-    (fp_line (start -1.2 8) (end 1.2 8) (layer F.SilkS) (width 0.15))
-    (fp_line (start 1.2 -10.25) (end 1.2 10.25) (layer F.SilkS) (width 0.15))
-    (fp_line (start 1.2 10.25) (end -1.2 10.25) (layer F.SilkS) (width 0.15))
-    (fp_line (start -1.2 10.25) (end -1.2 -10.25) (layer F.SilkS) (width 0.15))
-    (fp_line (start -1.2 -10.25) (end 1.2 -10.25) (layer F.SilkS) (width 0.15))
-    (pad 1 smd rect (at -2.54 9) (size 2.29 0.89) (layers F.Cu F.Paste F.Mask)
-      (net 24 "Net-(H2-Pad1)"))
-    (pad 2 smd rect (at 2.54 7) (size 2.29 0.89) (layers F.Cu F.Paste F.Mask)
-      (net 26 "Net-(H2-Pad2)"))
-    (pad 3 smd rect (at -2.54 5) (size 2.29 0.89) (layers F.Cu F.Paste F.Mask)
-      (net 27 "Net-(H2-Pad3)"))
-    (pad 4 smd rect (at 2.54 3) (size 2.29 0.89) (layers F.Cu F.Paste F.Mask)
-      (net 28 "Net-(H2-Pad4)"))
-    (pad 5 smd rect (at -2.54 1) (size 2.29 0.89) (layers F.Cu F.Paste F.Mask)
-      (net 29 "Net-(H2-Pad5)"))
-    (pad 6 smd rect (at 2.54 -1) (size 2.29 0.89) (layers F.Cu F.Paste F.Mask)
-      (net 30 "Net-(H2-Pad6)"))
-    (pad 7 smd rect (at -2.54 -3) (size 2.29 0.89) (layers F.Cu F.Paste F.Mask)
-      (net 31 "Net-(H2-Pad7)"))
-    (pad 8 smd rect (at 2.54 -5) (size 2.29 0.89) (layers F.Cu F.Paste F.Mask)
-      (net 32 "Net-(H2-Pad8)"))
-    (pad 9 smd rect (at -2.54 -7) (size 2.29 0.89) (layers F.Cu F.Paste F.Mask)
-      (net 33 "Net-(H2-Pad9)"))
-    (pad 10 smd rect (at 2.54 -9) (size 2.29 0.89) (layers F.Cu F.Paste F.Mask)
-      (net 25 "Net-(H2-Pad10)"))
   )
   (module _MUSB_SM0603_Resistor (layer F.Cu)
@@
       (net 11 "Net-(D1-Pad2)"))
   )
+  (module _MUSB_:_MUSB-FEMALE-HEADER-NPPN101BFLD-RC-Pin1Right (layer F.Cu)
+    (at 137.5 114.004 180)
+    (fp_text reference H1 (at 2.55 9 180) (layer F.SilkS)
+      (effects (font (size 1 1) (thickness 0.15)))
+    )
+    (fp_text value XBeeLeftPins (at 0 11.57 180) (layer F.SilkS) hide
+      (effects (font (size 1 1) (thickness 0.15)))
+    )
+    (fp_line (start -1.2 8) (end 1.2 8) (layer F.SilkS) (width 0.15))
+    (fp_line (start 1.2 -10.25) (end 1.2 10.25) (layer F.SilkS) (width 0.15))
+    (fp_line (start 1.2 10.25) (end -1.2 10.25) (layer F.SilkS) (width 0.15))
+    (fp_line (start -1.2 10.25) (end -1.2 -10.25) (layer F.SilkS) (width 0.15))
+    (fp_line (start -1.2 -10.25) (end 1.2 -10.25) (layer F.SilkS) (width 0.15))
+    (pad 1 smd rect (at 2.54 9 180) (size 2.29 0.89) (layers F.Cu F.Paste F.Mask)
+      (net 6 BAT+))
+    (pad 2 smd rect (at -2.54 7 180) (size 2.29 0.89) (layers F.Cu F.Paste F.Mask)
+      (net 16 "Net-(H1-Pad2)"))
+    (pad 3 smd rect (at 2.54 5 180) (size 2.29 0.89) (layers F.Cu F.Paste F.Mask)
+      (net 17 "Net-(H1-Pad3)"))
+    (pad 4 smd rect (at -2.54 3 180) (size 2.29 0.89) (layers F.Cu F.Paste F.Mask)
+      (net 18 "Net-(H1-Pad4)"))
+    (pad 5 smd rect (at 2.54 1 180) (size 2.29 0.89) (layers F.Cu F.Paste F.Mask)
+      (net 19 "Net-(H1-Pad5)"))
+    (pad 6 smd rect (at -2.54 -1 180) (size 2.29 0.89) (layers F.Cu F.Paste F.Mask)
+      (net 20 "Net-(H1-Pad6)"))
+    (pad 7 smd rect (at 2.54 -3 180) (size 2.29 0.89) (layers F.Cu F.Paste F.Mask)
+      (net 21 "Net-(H1-Pad7)"))
+    (pad 8 smd rect (at -2.54 -5 180) (size 2.29 0.89) (layers F.Cu F.Paste F.Mask)
+      (net 22 "Net-(H1-Pad8)"))
+    (pad 9 smd rect (at 2.54 -7 180) (size 2.29 0.89) (layers F.Cu F.Paste F.Mask)
+      (net 23 "Net-(H1-Pad9)"))
+    (pad 10 smd rect (at -2.54 -9 180) (size 2.29 0.89) (layers F.Cu F.Paste F.Mask)
+      (net 7 GND))
+  )
+  (module _MUSB_:_MUSB-FEMALE-HEADER-NPPN101BFLC-RC-Pin1Left (layer F.Cu)
+    (at 159.502 114.004)
+    (fp_text reference H2 (at -2.55 9.05) (layer F.SilkS)
+      (effects (font (size 1 1) (thickness 0.15)))
+    )
+    (fp_text value XBeeRightPins (at 0 11.57) (layer F.SilkS) hide
+      (effects (font (size 1 1) (thickness 0.15)))
+    )
+    (fp_line (start -1.2 8) (end 1.2 8) (layer F.SilkS) (width 0.15))
+    (fp_line (start 1.2 -10.25) (end 1.2 10.25) (layer F.SilkS) (width 0.15))
+    (fp_line (start 1.2 10.25) (end -1.2 10.25) (layer F.SilkS) (width 0.15))
+    (fp_line (start -1.2 10.25) (end -1.2 -10.25) (layer F.SilkS) (width 0.15))
+    (fp_line (start -1.2 -10.25) (end 1.2 -10.25) (layer F.SilkS) (width 0.15))
+    (pad 1 smd rect (at -2.54 9) (size 2.29 0.89) (layers F.Cu F.Paste F.Mask)
+      (net 24 "Net-(H2-Pad1)"))
+    (pad 2 smd rect (at 2.54 7) (size 2.29 0.89) (layers F.Cu F.Paste F.Mask)
+      (net 26 "Net-(H2-Pad2)"))
+    (pad 3 smd rect (at -2.54 5) (size 2.29 0.89) (layers F.Cu F.Paste F.Mask)
+      (net 27 "Net-(H2-Pad3)"))
+    (pad 4 smd rect (at 2.54 3) (size 2.29 0.89) (layers F.Cu F.Paste F.Mask)
+      (net 28 "Net-(H2-Pad4)"))
+    (pad 5 smd rect (at -2.54 1) (size 2.29 0.89) (layers F.Cu F.Paste F.Mask)
+      (net 29 "Net-(H2-Pad5)"))
+    (pad 6 smd rect (at 2.54 -1) (size 2.29 0.89) (layers F.Cu F.Paste F.Mask)
+      (net 30 "Net-(H2-Pad6)"))
+    (pad 7 smd rect (at -2.54 -3) (size 2.29 0.89) (layers F.Cu F.Paste F.Mask)
+      (net 31 "Net-(H2-Pad7)"))
+    (pad 8 smd rect (at 2.54 -5) (size 2.29 0.89) (layers F.Cu F.Paste F.Mask)
+      (net 32 "Net-(H2-Pad8)"))
+    (pad 9 smd rect (at -2.54 -7) (size 2.29 0.89) (layers F.Cu F.Paste F.Mask)
+      (net 33 "Net-(H2-Pad9)"))
+    (pad 10 smd rect (at 2.54 -9) (size 2.29 0.89) (layers F.Cu F.Paste F.Mask)
+      (net 25 "Net-(H2-Pad10)"))
+  )
   (gr_text M9Design.co (at 153.58 137.5 270) (layer F.SilkS)
